Commit message: gazebo no model

File: description/gazebo_control.xacro (robot description, xacro)
@@ -3,5 +3,7 @@
   <!-- Gazebo ROS Control Plugin -->
   <gazebo>
-    <plugin name="diff_drive" filename="libgazebo_ros_diff_drive.so"/>
+    <plugin name="gazebo_ros_control" filename="libgazebo_ros_control.so">
+      <robotNamespace>/</robotNamespace>
+    </plugin>
   </gazebo>
   <!-- Transmission and Controller Interfaces for Each Joint -->
@@ -24,3 +26,24 @@
   <xacro:transmission_interface joint_name="wrist"/>
   <xacro:transmission_interface joint_name="joint_end_effector"/>
+  <!-- Optional: Add physics parameters for each joint link -->
+  <gazebo reference="base_link">
+    <kp>100.0</kp>
+    <kd>1.0</kd>
+  </gazebo>
+  <gazebo reference="shoulder_link">
+    <kp>100.0</kp>
+    <kd>1.0</kd>
+  </gazebo>
+  <gazebo reference="elbow_link">
+    <kp>100.0</kp>
+    <kd>1.0</kd>
+  </gazebo>
+  <gazebo reference="wrist_link">
+    <kp>100.0</kp>
+    <kd>1.0</kd>
+  </gazebo>
+  <gazebo reference="end_effector_link">
+    <kp>100.0</kp>
+    <kd>1.0</kd>
+  </gazebo>
 </robot>

File: description/robot.urdf.xacro (robot description, xacro)
@@ -3,9 +3,3 @@
     <xacro:include filename="robot_core.xacro" />
     <xacro:include filename="gazebo_control.xacro" />
-    <!-- ROS Control Plugin -->
-    <gazebo>
-        <plugin name="gazebo_ros_control" filename="libgazebo_ros_control.so">
-        <robotNamespace>/</robotNamespace>
-        </plugin>
-    </gazebo>
 </robot>

File: description/robot_core.xacro (robot description, xacro)
@@ -46,4 +46,7 @@
     </xacro:inertial_cylinder>
   </link>
+  <gazebo reference="link_1">
+    <material>Gazebo/black</material>
+  </gazebo>
   <!-- ARM 1 (500mm) -->
   <joint name="shoulder" type="revolute">
@@ -72,4 +75,7 @@
     </xacro:inertial_cylinder>
   </link>
+  <gazebo reference="upper_arm">
+    <material>Gazebo/blue</material>
+  </gazebo>
   <!-- ARM 2 (400mm) -->
   <joint name="elbow" type="revolute">
@@ -98,4 +104,7 @@
     </xacro:inertial_cylinder>
   </link>
+  <gazebo reference="fore_arm">
+    <material>Gazebo/gray</material>
+  </gazebo>
   <!-- ARM 3 (100mm) -->
   <joint name="wrist" type="revolute">
@@ -124,4 +133,7 @@
     </xacro:inertial_cylinder>
   </link>
+  <gazebo reference="hand">
+    <material>Gazebo/white</material>
+  </gazebo>
   <!-- END EFFECTOR (360-degree rotation) -->
   <joint name="joint_end_effector" type="continuous">
@@ -149,3 +161,6 @@
     </xacro:inertial_cylinder>
   </link>
+  <gazebo reference="fingers">
+    <material>Gazebo/orange</material>
+  </gazebo>
 </robot>

Commit message: Gazebo Fixed

File: description/gazebo_control.xacro (robot description, xacro)
@@ -3,5 +3,6 @@
   <!-- Gazebo ROS Control Plugin -->
   <gazebo>
-    <plugin name="gazebo_ros_control" filename="libgazebo_ros_control.so">
+    <plugin name="gazebo_ros_control" filename="libgazebo_ros_factory.so">
+    <!-- <plugin name="gazebo_ros_factory" filename="libgazebo_ros_factory.so"> -->
       <robotNamespace>/</robotNamespace>
     </plugin>

File: description/robot_core.xacro (robot description, xacro)
@@ -19,5 +19,20 @@
     </material>
   <!-- BASE LINK -->
-  <link name="base_link">
+    <link name="base_link">
+      <visual>
+        <geometry>
+          <cylinder length="0.1" radius="0.2"/> <!-- Adjust dimensions as needed -->
+        </geometry>
+        <material name="orange"/>
+      </visual>
+      <collision>
+        <geometry>
+          <cylinder length="0.1" radius="0.2"/>
+        </geometry>
+      </collision>
+      <inertial>
+        <mass value="1.0"/>
+        <inertia ixx="0.01" ixy="0" ixz="0" iyy="0.01" iyz="0" izz="0.01"/>
+      </inertial>
     </link>
   <!-- BASE ROTATION JOINT (360 degrees) -->
